Commit message: added aruco models

File: swarm_description/models/agent3/bot.urdf.xacro (robot description, xacro)
@@ -40,5 +40,6 @@
 		<visual>
 			<geometry>
-				<cylinder length="0.12" radius="0.1"/>
+				<!--<cylinder length="0.12" radius="0.1"/>-->
+				<mesh filename="package://swarm_description/models/TagModels/tag3/apriltag_work.dae"/>
 			</geometry>
 			<origin rpy="0 0 0" xyz="0 0 0.085"/>
