Commit message: added models and detection script

File: swarm_description/models/agent0/bot.urdf.xacro (robot description, xacro)
@@ -41,5 +41,5 @@
 			<geometry>
 				<!--<cylinder length="0.12" radius="0.1"/>-->
-				<mesh filename="package://swarm_description/models/TagModels/tag0/apriltag_work.dae"/>
+				<mesh filename="package://swarm_description/models/agent0/meshes/apriltag_work.dae"/>
 			</geometry>
 			<origin rpy="0 0 0" xyz="0 0 0.085"/>

File: swarm_description/models/agent1/bot.urdf.xacro (robot description, xacro)
@@ -41,5 +41,5 @@
 			<geometry>
 				<!--<cylinder length="0.12" radius="0.1"/>-->
-				<mesh filename="package://swarm_description/models/TagModels/tag1/apriltag_work.dae"/>
+				<mesh filename="package://swarm_description/models/agent1/meshes/apriltag_work.dae"/>
 			</geometry>
 			<origin rpy="0 0 0" xyz="0 0 0.085"/>

File: swarm_description/models/agent10/bot.urdf.xacro (robot description, xacro)
@@ -41,5 +41,5 @@
 			<geometry>
 				<!--<cylinder length="0.12" radius="0.1"/>-->
-				<mesh filename="package://swarm_description/models/TagModels/tag10/apriltag_work.dae"/>
+				<mesh filename="package://swarm_description/models/agent10/meshes/apriltag_work.dae"/>
 			</geometry>
 			<origin rpy="0 0 0" xyz="0 0 0.085"/>

File: swarm_description/models/agent2/bot.urdf.xacro (robot description, xacro)
@@ -41,5 +41,5 @@
 			<geometry>
 				<!--<cylinder length="0.12" radius="0.1"/>-->
-				<mesh filename="package://swarm_description/models/TagModels/tag2/apriltag_work.dae"/>
+				<mesh filename="package://swarm_description/models/agent2/meshes/apriltag_work.dae"/>
 			</geometry>
 			<origin rpy="0 0 0" xyz="0 0 0.085"/>

File: swarm_description/models/agent3/bot.urdf.xacro (robot description, xacro)
@@ -41,5 +41,5 @@
 			<geometry>
 				<!--<cylinder length="0.12" radius="0.1"/>-->
-				<mesh filename="package://swarm_description/models/TagModels/tag3/apriltag_work.dae"/>
+				<mesh filename="package://swarm_description/models/agent3/meshes/apriltag_work.dae"/>
 			</geometry>
 			<origin rpy="0 0 0" xyz="0 0 0.085"/>

File: swarm_description/models/agent4/bot.urdf.xacro (robot description, xacro)
@@ -41,5 +41,5 @@
 			<geometry>
 				<!--<cylinder length="0.12" radius="0.1"/>-->
-				<mesh filename="package://swarm_description/models/TagModels/tag4/apriltag_work.dae"/>
+				<mesh filename="package://swarm_description/models/agent4/meshes/apriltag_work.dae"/>
 			</geometry>
 			<origin rpy="0 0 0" xyz="0 0 0.085"/>

File: swarm_description/models/agent5/bot.urdf.xacro (robot description, xacro)
@@ -41,5 +41,5 @@
 			<geometry>
 				<!--<cylinder length="0.12" radius="0.1"/>-->
-				<mesh filename="package://swarm_description/models/TagModels/tag5/apriltag_work.dae"/>
+				<mesh filename="package://swarm_description/models/agent5/meshes/apriltag_work.dae"/>
 			</geometry>
 			<origin rpy="0 0 0" xyz="0 0 0.085"/>

File: swarm_description/models/agent6/bot.urdf.xacro (robot description, xacro)
@@ -41,5 +41,5 @@
 			<geometry>
 				<!--<cylinder length="0.12" radius="0.1"/>-->
-				<mesh filename="package://swarm_description/models/TagModels/tag6/apriltag_work.dae"/>
+				<mesh filename="package://swarm_description/models/agent6/meshes/apriltag_work.dae"/>
 			</geometry>
 			<origin rpy="0 0 0" xyz="0 0 0.085"/>

File: swarm_description/models/agent7/bot.urdf.xacro (robot description, xacro)
@@ -41,5 +41,5 @@
 			<geometry>
 				<!--<cylinder length="0.12" radius="0.1"/>-->
-				<mesh filename="package://swarm_description/models/TagModels/tag7/apriltag_work.dae"/>
+				<mesh filename="package://swarm_description/models/agent7/meshes/apriltag_work.dae"/>
 			</geometry>
 			<origin rpy="0 0 0" xyz="0 0 0.085"/>

File: swarm_description/models/agent8/bot.urdf.xacro (robot description, xacro)
@@ -41,5 +41,5 @@
 			<geometry>
 				<!--<cylinder length="0.12" radius="0.1"/>-->
-				<mesh filename="package://swarm_description/models/TagModels/tag8/apriltag_work.dae"/>
+				<mesh filename="package://swarm_description/models/agent8/meshes/apriltag_work.dae"/>
 			</geometry>
 			<origin rpy="0 0 0" xyz="0 0 0.085"/>

File: swarm_description/models/agent9/bot.urdf.xacro (robot description, xacro)
@@ -41,5 +41,5 @@
 			<geometry>
 				<!--<cylinder length="0.12" radius="0.1"/>-->
-				<mesh filename="package://swarm_description/models/TagModels/tag9/apriltag_work.dae"/>
+				<mesh filename="package://swarm_description/models/agent9/meshes/apriltag_work.dae"/>
 			</geometry>
 			<origin rpy="0 0 0" xyz="0 0 0.085"/>
